Commit message: Modified files

File: urdf/my_robot_integration.xacro (robot description, xacro)
@@ -5,11 +5,11 @@
 	<!-- Include Robot's urdf filepath -->
 	<!-- Include Lidar's urdf filepath -->
-	<xacro:include filename="mobile_robot.urdf"/>
-	<xacro:include filename="ydlidar.urdf"/>
+	<xacro:include filename="$(find mobile_robot)/urdf/mobile_robot.urdf"/>
+	<xacro:include filename="$(find mobile_robot)/urdf/ydlidar.urdf"/>
 <!-- Add your gazebo sensors here -->
 <gazebo reference="base_laser">
 		<!-- <gravity>true</gravity> -->
 		<!-- Gazebo has fixed set of Sensors types. Check them out here <> -->
-		<sensor name="lidar" type="ray">
+		<sensor name="laser" type="ray">
 			<!-- Add in your sensor characteristics -->
 			<pose> 0 0 0 0 0 0 </pose>
@@ -39,5 +39,5 @@
             <plugin name="gazebo_ros_head_hokuyo_controller" filename="libgazebo_ros_laser.so">
             	<!-- Use topic name as /my_robot/scan -->
-				<topicName>/mobile_robot</topicName>
+				<topicName>/mobile_robot/scan</topicName>
 				<frameName>laser_frame</frameName>
 			</plugin>
@@ -75,5 +75,5 @@
   <parent link="base_link"/>
   <child link="base_laser"/>
-  <origin xyz="0 0 0.5" rpy="0 0 0"/>
+  <origin xyz="0 0 0.44" rpy="90 0 0"/>
 </joint>
 </robot>

File: urdf/robot_plus_lidar.urdf (robot description, URDF)
Before this commit: robot mobile_robot, 12 links, 11 joints
Joints:
- joint lidar_joint: origin xyz=0 0 0.5 rpy=0 0 0 -> xyz=0 0 0.35 rpy=0 0 0
