Commit message: fixed axis error for front right wheel

File: urdf/mobile_robot.urdf (robot description, URDF)
Before this commit: robot mobile_robot, 9 links, 8 joints
Joints:
- joint front_right_wheel_shaft_joint: axis 0 0 0 -> 1 0 0

Commit message: added lidar urdf and xml files

File: urdf/mobile_robot.urdf (robot description, URDF)
Before this commit: robot mobile_robot, 9 links, 8 joints
Links:
- added link dummy_link
Joints:
- added joint dummy_joint: type fixed, parent dummy_link, child base_link, origin xyz=0 0 0 rpy=0 0 0, axis 0 0 0

File: urdf/ydlidar.urdf (robot description, URDF)
Before this commit: robot ydlidar, 2 links, 1 joints
Links:
- link base_laser: geometry collision mesh filename=package://mobile_robot/meshes/ydlidar.dae; visual mesh filename=package://mobile_robot/meshes/ydlidar.dae
- link laser_frame: geometry collision mesh filename=package://mobile_robot/meshes/ydlidar.dae; visual mesh filename=package://mobile_robot/meshes/ydlidar.dae

Commit message: Updated meshed and urdf after adding shaft axis

File: urdf/mobile_robot.urdf (robot description, URDF)
Before this commit: robot mobile_robot, 10 links, 9 joints
Links:
- removed link front_left_wheel_shaft
- removed link front_right_wheel_shaft
- removed link rear_left_wheel_shaft
- removed link rear_right_wheel_shaft
- added link front_left_shaft, mass 0.535359728660285; collision mesh filename=package://mobile_robot/meshes/front_left_shaft.STL; visual mesh filename=package://mobile_robot/meshes/front_left_shaft.STL
- added link front_right_shaft, mass 0.535359914923846; collision mesh filename=package://mobile_robot/meshes/front_right_shaft.STL; visual mesh filename=package://mobile_robot/meshes/front_right_shaft.STL
- added link rear_wheel_shaft, mass 1.02790122650355; collision mesh filename=package://mobile_robot/meshes/rear_wheel_shaft.STL; visual mesh filename=package://mobile_robot/meshes/rear_wheel_shaft.STL
- link base_link: mass 68.3202619212701 -> 30.1147830562474
- link front_left_wheel: mass 0.898923461702659 -> 0.627305726641922
- link front_right_wheel: mass 0.898923461702655 -> 0.627305726641922
- link rear_left_wheel: mass 0.898923461702657 -> 0.627305726641922
- link rear_right_wheel: mass 0.898923461702656 -> 0.627305726641923
Joints:
- removed joint front_left_wheel_shaft_joint
- removed joint front_right_wheel_shaft_joint
- removed joint rear_left_wheel_shaft_joint
- removed joint rear_right_wheel_shaft_joint
- added joint front_left_shaft_joint: type continuous, parent base_link, child front_left_shaft, origin xyz=0.254 0.1016 0.10414 rpy=0 0 1.5708, axis 0 0 1, limit lower=0 upper=0 effort=0 velocity=0
- added joint front_right_shaft_joint: type continuous, parent base_link, child front_right_shaft, origin xyz=0.254 -0.1016 0.10414 rpy=0 0 1.5708, axis 0 0 1, limit lower=0 upper=0 effort=0 velocity=0
- added joint rear_wheel_shaft_joint: type continuous, parent base_link, child rear_wheel_shaft, origin xyz=-0.254 -0.254 0.10414 rpy=-1.5708 0 0, axis 0 0 1
- joint front_left_wheel_joint: axis -0.00273683970937426 0 -0.999996254847189 -> 0.019056 0 0.99982; origin xyz=0 0 0 rpy=0 0 0 -> xyz=0.15162 -0.015401 0 rpy=-1.5708 0 -1.5708; parent front_left_wheel_shaft -> front_left_shaft
- joint front_right_wheel_joint: axis -0.00273683970937426 0 -0.999996254847189 -> 0.019056 0 0.99982; origin xyz=0 0 0 rpy=0 0 0 -> xyz=-0.15229 -0.0057359 0 rpy=-1.5708 0 -1.5708; parent front_right_wheel_shaft -> front_right_shaft
- joint rear_left_wheel_joint: origin xyz=0 0 0 rpy=0 0 0 -> xyz=0 0 0.508 rpy=0 0 0; parent rear_left_wheel_shaft -> rear_wheel_shaft
- joint rear_right_wheel_joint: parent rear_right_wheel_shaft -> rear_wheel_shaft

File: urdf/my_robot_integration.xacro (robot description, xacro)
@@ -75,5 +75,5 @@
   <parent link="base_link"/>
   <child link="base_laser"/>
-  <origin xyz="0 0 0.44" rpy="90 0 0"/>
+  <origin xyz="0 0 0.3" rpy="0 0 0"/>
 </joint>
 </robot>

File: urdf/robot_plus_lidar.urdf (robot description, URDF)
Before this commit: robot mobile_robot, 12 links, 11 joints
Links:
- removed link front_left_wheel_shaft
- removed link front_right_wheel_shaft
- removed link rear_left_wheel_shaft
- removed link rear_right_wheel_shaft
- added link front_left_shaft, mass 0.535359728660285; collision mesh filename=package://mobile_robot/meshes/front_left_shaft.STL; visual mesh filename=package://mobile_robot/meshes/front_left_shaft.STL
- added link front_right_shaft, mass 0.535359914923846; collision mesh filename=package://mobile_robot/meshes/front_right_shaft.STL; visual mesh filename=package://mobile_robot/meshes/front_right_shaft.STL
- added link rear_wheel_shaft, mass 1.02790122650355; collision mesh filename=package://mobile_robot/meshes/rear_wheel_shaft.STL; visual mesh filename=package://mobile_robot/meshes/rear_wheel_shaft.STL
- link base_link: mass 68.3202619212701 -> 30.1147830562474
- link front_left_wheel: mass 0.898923461702659 -> 0.627305726641922
- link front_right_wheel: mass 0.898923461702655 -> 0.627305726641922
- link rear_left_wheel: mass 0.898923461702657 -> 0.627305726641922
- link rear_right_wheel: mass 0.898923461702656 -> 0.627305726641923
Joints:
- removed joint front_left_wheel_shaft_joint
- removed joint front_right_wheel_shaft_joint
- removed joint rear_left_wheel_shaft_joint
- removed joint rear_right_wheel_shaft_joint
- added joint front_left_shaft_joint: type continuous, parent base_link, child front_left_shaft, origin xyz=0.254 0.1016 0.10414 rpy=0 0 1.5708, axis 0 0 1, limit lower=0 upper=0 effort=0 velocity=0
- added joint front_right_shaft_joint: type continuous, parent base_link, child front_right_shaft, origin xyz=0.254 -0.1016 0.10414 rpy=0 0 1.5708, axis 0 0 1, limit lower=0 upper=0 effort=0 velocity=0
- added joint rear_wheel_shaft_joint: type continuous, parent base_link, child rear_wheel_shaft, origin xyz=-0.254 -0.254 0.10414 rpy=-1.5708 0 0, axis 0 0 1
- joint front_left_wheel_joint: axis -0.00273683970937426 0 -0.999996254847189 -> 0.019056 0 0.99982; origin xyz=0 0 0 rpy=0 0 0 -> xyz=0.15162 -0.015401 0 rpy=-1.5708 0 -1.5708; parent front_left_wheel_shaft -> front_left_shaft
- joint front_right_wheel_joint: axis -0.00273683970937426 0 -0.999996254847189 -> 0.019056 0 0.99982; origin xyz=0 0 0 rpy=0 0 0 -> xyz=-0.15229 -0.0057359 0 rpy=-1.5708 0 -1.5708; parent front_right_wheel_shaft -> front_right_shaft
- joint lidar_joint: origin xyz=0 0 0.35 rpy=0 0 0 -> xyz=0 0 0.44 rpy=90 0 0
- joint rear_left_wheel_joint: origin xyz=0 0 0 rpy=0 0 0 -> xyz=0 0 0.508 rpy=0 0 0; parent rear_left_wheel_shaft -> rear_wheel_shaft
- joint rear_right_wheel_joint: parent rear_right_wheel_shaft -> rear_wheel_shaft

Commit message: Updated urdf files

File: urdf/mobile_robot.urdf (robot description, URDF)
Before this commit: robot mobile_robot, 9 links, 8 joints
Joints:
- joint front_left_shaft_joint: limit lower=0 upper=0 effort=0 velocity=0 -> lower=-3.14 upper=3.14 effort=10 velocity=10000
- joint front_right_shaft_joint: limit lower=0 upper=0 effort=0 velocity=0 -> lower=-3.14 upper=3.14 effort=10 velocity=10000

File: urdf/my_robot_integration.xacro (robot description, xacro)
@@ -75,5 +75,5 @@
   <parent link="base_link"/>
   <child link="base_laser"/>
-  <origin xyz="0 0 0.3" rpy="0 0 0"/>
+  <origin xyz="0 0 0.27" rpy="0 0 0"/>
 </joint>
 </robot>
